File: hardware/Breakout/breakout.brd (EAGLE design)
At the start: 101.6 x 86.3 mm, 44 parts, among them CON2 LED2, CON5 LED1, IC1 24AA04SN, IC2 MAX490CSA, IC3 MAX490CSA, IC4 PCA9685, X1 VISCA, X2 RS485, X3 JOYSTICK, X4 SLIDER

Commit message: Breakout board fixes
Pullups for I2C2, power cycle external boards.
Parts:
- added C1, C3, C4: 100nF, SparkFun:0603-CAP
- added C5, C6: 1u, resistor:C0805
- added R23, R24: 4.7K, resistor:R0603
- added R25, R26: 1K, resistor:R0603
- added U$1, U$2: IRLML6402, IRLML6402:SOT-23
- renumbered SV1 to DISPLAY
Connections:
- new net N$13: C5.1, DISPLAY.2, U$2.3
- new net N$3: C5.2, R25.1, U$2.1
- new net N$6: C6.2, R26.1, U$1.1
- new net N$8: BI8_SERIAL1.2, BI8_SERIAL2.2, C6.1, U$1.3
- net GND: now also C1.2, C3.2, C4.2
- net I2C2_SCL: now also R23.2
- net I2C2_SDA: now also R24.2
- net PG0: now also R26.2
- net PG1: now also R25.2
- net VCC: now also C1.1, C3.1, C4.1, R23.1, R24.1, U$1.2, U$2.2; no longer BI8_SERIAL1.2, BI8_SERIAL2.2, DISPLAY.2
Routing:
- net PG0: track 0.00 -> 60.1 mm, vias 0 -> 1
- net VCC: track 368.1 -> 404.0 mm
- net N$8: track 0.00 -> 26.2 mm
- net PG1: track 0.00 -> 15.0 mm
- net N$13: track 0.00 -> 9.21 mm
- net N$6: track 0.00 -> 8.02 mm
- net N$3: track 0.00 -> 6.17 mm
- net GND: track 410.3 -> 414.6 mm, vias 3 -> 4
- net I2C2_SDA: track 76.7 -> 79.8 mm
- net I2C2_SCL: track 93.1 -> 94.9 mm
- net A4: track 106.0 -> 107.3 mm
- net A3: track 98.9 -> 99.7 mm
- net A2: track 96.5 -> 97.2 mm
Other:
- board text added: "10/2013"
- board text added: "SLIDER"
- board text removed: "07/2013"

Commit message: Pull-up for SPI2 MOSI (see UEXT on mainboard)
Parts:
- added R27: 47K, resistor:R0603
Connections:
- net GND: now also IC4.4
- net SPI1_MOSI: now also R27.2
- net VCC: now also R27.1; no longer IC4.4
Routing:
- net VCC: track 404.0 -> 413.0 mm
- net SPI1_MOSI: track 65.1 -> 69.6 mm
Changed lines of the file:
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@@
 <?xml version="1.0" encoding="utf-8"?>
 <!DOCTYPE eagle SYSTEM "eagle.dtd">
-<eagle version="6.5.0">
+<eagle version="6.4">
 <drawing>
 <settings>
@@
 <attribute name="VALUE" x="24.13" y="27.051" size="1.27" layer="27" rot="R90"/>
 </element>
+<element name="R27" library="resistor" package="R0603" value="47K" x="48.768" y="15.24" rot="R90"/>
 </elements>
 <signals>
@@
 <contactref element="C2" pad="1"/>
 <contactref element="IC4" pad="28"/>
-<contactref element="IC4" pad="4"/>
 <wire x1="55.5022" y1="47.853" x2="61.3378" y2="47.853" width="0.254" layer="1"/>
 <wire x1="54.763" y1="47.853" x2="54.61" y2="48.006" width="0.254" layer="1"/>
@@
 <wire x1="54.61" y1="48.387" x2="54.737" y2="48.514" width="0.254" layer="1"/>
 <wire x1="54.737" y1="48.514" x2="55.4912" y2="48.514" width="0.254" layer="1"/>
-<wire x1="55.4912" y1="48.514" x2="55.5022" y2="48.503" width="0.254" layer="1"/>
 <wire x1="79.375" y1="5.27" x2="79.375" y2="36.957" width="0.254" layer="16"/>
 <wire x1="79.375" y1="36.957" x2="80.01" y2="37.592" width="0.254" layer="16"/>
@@
 <wire x1="35.56" y1="9.144" x2="42.164" y2="9.144" width="0.254" layer="1"/>
 <wire x1="42.164" y1="9.144" x2="43.815" y2="7.493" width="0.254" layer="1"/>
-<wire x1="43.815" y1="7.493" x2="43.815" y2="5.07" width="0.254" layer="1"/>
+<wire x1="43.815" y1="7.493" x2="43.815" y2="7.366" width="0.254" layer="1"/>
+<wire x1="43.815" y1="7.366" x2="43.815" y2="5.07" width="0.254" layer="1"/>
 <wire x1="20.955" y1="77.851" x2="20.955" y2="78.73" width="0.254" layer="1"/>
 <wire x1="3.81" y1="44.14" x2="3.81" y2="49.784" width="0.254" layer="16"/>
@@
 <wire x1="50.448" y1="78.73" x2="52.06" y2="78.73" width="0.254" layer="16"/>
 <wire x1="52.06" y1="78.73" x2="52.07" y2="78.74" width="0.254" layer="16"/>
+<contactref element="R27" pad="1"/>
+<wire x1="48.768" y1="14.39" x2="48.768" y2="12.319" width="0.254" layer="1"/>
+<wire x1="48.768" y1="12.319" x2="43.815" y2="7.366" width="0.254" layer="1"/>
 <wire x1="21.082" y1="78.74" x2="20.955" y2="78.73" width="0" layer="19" extent="16-16"/>
 </signal>
@@
 <wire x1="38.735" y1="64.643" x2="38.735" y2="68.453" width="0.254" layer="1"/>
 <wire x1="38.735" y1="68.453" x2="42.418" y2="72.136" width="0.254" layer="1"/>
+<contactref element="IC4" pad="4"/>
+<wire x1="55.5022" y1="49.153" x2="55.5022" y2="48.503" width="0" layer="19" extent="1-1"/>
 </signal>
 <signal name="A1">
@@
 <wire x1="44.958" y1="29.464" x2="48.895" y2="25.527" width="0.254" layer="1"/>
 <wire x1="48.895" y1="25.527" x2="48.895" y2="20.51" width="0.254" layer="1"/>
+<contactref element="R27" pad="2"/>
+<wire x1="48.768" y1="16.09" x2="48.895" y2="16.09" width="0.254" layer="1"/>
+<wire x1="48.895" y1="16.09" x2="48.895" y2="20.51" width="0.254" layer="1"/>
 </signal>
 <signal name="SPI1_MISO">
